File: Room_Monitor_C6.kicad_sch (KiCad schematic)
At the start: 39 parts, among them J1 USB_C_Receptacle_USB2.0_16P, J3 FH34SRJ-24S-0.5SH_99_, Q1 AO3400A, SW1 SW_SPST, SW2 SW_SPST, U1 ESP32-C6-MINI-1/U, U2 SHT4x, U3 SCD43-D-R2, U4 USBLC6-2SC6, U6 TLV75733PDBV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

Commit message: Completed 4-layer PCB layout
Parts:
- added H1, H2, H3: MountingHole_Pad, MountingHole:MountingHole_2.2mm_M2_Pad, symbol Mechanical:MountingHole_Pad
- C1, C2, C3: footprint (none) -> Capacitor_SMD:C_0805_2012Metric
- C10, C11, C12, C13, C8, C9: value 1µF 25V -> 1µF 50V; footprint Capacitor_SMD:C_0805_2012Metric -> Capacitor_SMD:C_0603_1608Metric
- C14, C4, C5, C6, C7: footprint (none) -> Capacitor_SMD:C_0402_1005Metric
- C15: value 1µF 25V -> 1µF 50V
- J1: footprint (none) -> Connector_USB:USB_C_Receptacle_GCT_USB4105-xx-A_16P_TopMnt_Horizontal
- R1, R11, R2, R3, R4, R5, R6, R7, R8, R9: footprint (none) -> Resistor_SMD:R_0603_1608Metric
- R10: footprint Resistor_SMD:R_0402_1005Metric -> Resistor_SMD:R_0603_1608Metric
- SW1, SW2: footprint (none) -> Button_Switch_SMD:SW_SPST_SKQG_WithoutStem
- U7: footprint SS2040FL:SOD-123FL -> Diode_SMD:D_SOD-123F
Connections:
- net GND: now also H1.1, H2.1, H3.1
Other:
- moved on the sheet: C15
